Commit message: Both diff_drive launch files working

File: diff_drive/urdf/ddrive.urdf.xacro (robot description, xacro)
@@ -1,10 +1,13 @@
-<robot name="i_am_wheelyboy" xmlns:xacro="http://ros.org/wiki/xacro">
+<robot name="wheelyboy" xmlns:xacro="http://ros.org/wiki/xacro">
+    <xacro:include filename="ddrive.gazebo.xacro"/>
     <xacro:property name="ddrive_yaml" value="$(find diff_drive)/config/ddrive.yaml"/>
     <xacro:property name="ddrive_yaml_info" value="${load_yaml(ddrive_yaml)}"/>
-    <xacro:property name="L" value="${ddrive_yaml_info['Length']}"/>
-    <xacro:property name="W" value="${ddrive_yaml_info['Width']}"/>
-    <xacro:property name="H" value="${ddrive_yaml_info['Height']}"/>
-    <xacro:property name="WheelR" value="${ddrive_yaml_info['WheelR']}"/>
-    <xacro:property name="CasterR" value="${ddrive_yaml_info['CasterR']}"/>
+    <xacro:property name="L" value="${ddrive_yaml_info['body_length']}"/>
+    <xacro:property name="W" value="${ddrive_yaml_info['body_width']}"/>
+    <xacro:property name="H" value="${ddrive_yaml_info['body_height']}"/>
+    <xacro:property name="WheelR" value="${ddrive_yaml_info['wheel_radius']}"/>
+    <xacro:property name="WheelW" value="${ddrive_yaml_info['wheel_width']}"/>
+    <xacro:property name="CasterR" value="${ddrive_yaml_info['caster_radius']}"/>
+    <xacro:property name="CasterW" value="${ddrive_yaml_info['caster_width']}"/>
     <xacro:property name="PI" value="3.141592653"/>
     <link name="base_link"/>
@@ -53,5 +56,5 @@
             <origin xyz="0 0 0" rpy="0 ${PI/2} ${PI/2}"/>
             <geometry>
-                <cylinder length="0.1" radius="${WheelR}"/>
+                <cylinder length="${WheelW}" radius="${WheelR}"/>
             </geometry>
             <material name="yellow">
@@ -60,7 +63,7 @@
         </visual>
         <collision>
-            <origin xyz="0 0 0" rpy="0 0 0"/>
+            <origin xyz="0 0 0" rpy="0 ${PI/2} ${PI/2}"/>
             <geometry>
-                <cylinder length="0.1" radius="${WheelR}"/>
+                <cylinder length="${WheelW}" radius="${WheelR}"/>
             </geometry>
         </collision>
@@ -68,6 +71,6 @@
           <origin xyz="0 0 0" rpy="0 0 0"/>
           <mass value="1"/>
-          <inertia ixx="${(0.1*0.1/12) + (WheelR*WheelR/4)}" ixy="0" ixz="0"
-                     iyy="${(0.1*0.1/12) + (WheelR*WheelR/4)}" iyz="0"
+          <inertia ixx="${(WheelW*WheelW/12) + (WheelR*WheelR/4)}" ixy="0" ixz="0"
+                     iyy="${(WheelW*WheelW/12) + (WheelR*WheelR/4)}" iyz="0"
                      izz="${(WheelR*WheelR/2)}"/>
         </inertial>
@@ -77,5 +80,5 @@
             <origin xyz="0 0 0" rpy="0 ${PI/2} ${PI/2}"/>
             <geometry>
-                <cylinder length="0.1" radius="${WheelR}"/>
+                <cylinder length="${WheelW}" radius="${WheelR}"/>
             </geometry>
             <material name="yellow">
@@ -84,7 +87,7 @@
         </visual>
         <collision>
-            <origin xyz="0 0 0" rpy="0 0 0"/>
+            <origin xyz="0 0 0" rpy="0 ${PI/2} ${PI/2}"/>
             <geometry>
-                <cylinder length="0.1" radius="${WheelR}"/>
+                <cylinder length="${WheelW}" radius="${WheelR}"/>
             </geometry>
         </collision>
@@ -92,6 +95,6 @@
           <origin xyz="0 0 0" rpy="0 0 0"/>
           <mass value="1"/>
-          <inertia ixx="${(0.1*0.1/12) + (WheelR*WheelR/4)}" ixy="0" ixz="0"
-                     iyy="${(0.1*0.1/12) + (WheelR*WheelR/4)}" iyz="0"
+          <inertia ixx="${(WheelW*WheelW/12) + (WheelR*WheelR/4)}" ixy="0" ixz="0"
+                     iyy="${(WheelW*WheelW/12) + (WheelR*WheelR/4)}" iyz="0"
                      izz="${(WheelR*WheelR/2)}"/>
         </inertial>
@@ -113,5 +116,5 @@
             <origin xyz="0 0 0" rpy="0 ${PI/2} ${PI/2}"/>
             <geometry>
-                <cylinder length="0.1" radius="${CasterR}"/>
+                <cylinder length="${CasterW}" radius="${CasterR}"/>
             </geometry>
             <material name="yellow">
@@ -122,5 +125,5 @@
             <origin xyz="0 0 0" rpy="0 0 0"/>
             <geometry>
-                <cylinder length="0.1" radius="${CasterR}"/>
+                <cylinder length="${CasterW}" radius="${CasterR}"/>
             </geometry>
         </collision>
@@ -128,6 +131,6 @@
           <origin xyz="0 0 0" rpy="0 0 0"/>
           <mass value="1"/>
-          <inertia ixx="${(0.1*0.1/12) + (CasterR*CasterR/4)}" ixy="0" ixz="0"
-                     iyy="${(0.1*0.1/12) + (CasterR*CasterR/4)}" iyz="0"
+          <inertia ixx="${(CasterW*CasterW/12) + (CasterR*CasterR/4)}" ixy="0" ixz="0"
+                     iyy="${(CasterW*CasterW/12) + (CasterR*CasterR/4)}" iyz="0"
                      izz="${(CasterR*CasterR/2)}"/>
         </inertial>
@@ -137,5 +140,5 @@
             <origin xyz="0 0 0" rpy="0 ${PI/2} ${PI/2}"/>
             <geometry>
-                <cylinder length="0.1" radius="${CasterR}"/>
+                <cylinder length="${CasterW}" radius="${CasterR}"/>
             </geometry>
             <material name="yellow">
@@ -146,5 +149,5 @@
             <origin xyz="0 0 0" rpy="0 0 0"/>
             <geometry>
-                <cylinder length="0.1" radius="${CasterR}"/>
+                <cylinder length="${CasterW}" radius="${CasterR}"/>
             </geometry>
         </collision>
@@ -152,7 +155,7 @@
           <origin xyz="0 0 0" rpy="0 0 0"/>
           <mass value="1"/>
-          <inertia ixx="${(0.1*0.1/12) + (WheelR*WheelR/4)}" ixy="0" ixz="0"
-                     iyy="${(0.1*0.1/12) + (WheelR*WheelR/4)}" iyz="0"
-                     izz="${(WheelR*WheelR/2)}"/>
+          <inertia ixx="${(CasterW*CasterW/12) + (CasterR*CasterR/4)}" ixy="0" ixz="0"
+                     iyy="${(CasterW*CasterW/12) + (CasterR*CasterR/4)}" iyz="0"
+                     izz="${(CasterR*CasterR/2)}"/>
         </inertial>
     </link>

Commit message: Robot (mostly) successfully flips!

File: diff_drive/urdf/ddrive.urdf.xacro (robot description, xacro)
@@ -70,5 +70,5 @@
         <inertial>
           <origin xyz="0 0 0" rpy="0 0 0"/>
-          <mass value="1"/>
+          <mass value="10"/>
           <inertia ixx="${(WheelW*WheelW/12) + (WheelR*WheelR/4)}" ixy="0" ixz="0"
                      iyy="${(WheelW*WheelW/12) + (WheelR*WheelR/4)}" iyz="0"
@@ -94,5 +94,5 @@
         <inertial>
           <origin xyz="0 0 0" rpy="0 0 0"/>
-          <mass value="1"/>
+          <mass value="10"/>
           <inertia ixx="${(WheelW*WheelW/12) + (WheelR*WheelR/4)}" ixy="0" ixz="0"
                      iyy="${(WheelW*WheelW/12) + (WheelR*WheelR/4)}" iyz="0"
@@ -130,5 +130,5 @@
         <inertial>
           <origin xyz="0 0 0" rpy="0 0 0"/>
-          <mass value="1"/>
+          <mass value="0.5"/>
           <inertia ixx="${(CasterW*CasterW/12) + (CasterR*CasterR/4)}" ixy="0" ixz="0"
                      iyy="${(CasterW*CasterW/12) + (CasterR*CasterR/4)}" iyz="0"
@@ -154,5 +154,5 @@
         <inertial>
           <origin xyz="0 0 0" rpy="0 0 0"/>
-          <mass value="1"/>
+          <mass value="0.5"/>
           <inertia ixx="${(CasterW*CasterW/12) + (CasterR*CasterR/4)}" ixy="0" ixz="0"
                      iyy="${(CasterW*CasterW/12) + (CasterR*CasterR/4)}" iyz="0"
